File: PBJ_EU/PBJ_EU.kicad_sch (KiCad schematic)
At the start: 88 parts, among them J1 Molex_47257, J2 Molex_47257, J3 Molex_47257, J4 Molex_47257, J5 Conn_02x05_Odd_Even, J6 Conn_02x08_Odd_Even_Female, J7 Conn_02x05_Odd_Even, SW1 SW_SPDT, SW2 SW_SPDT, SW3 SW_DPST, SW4 SW_SPDT, U1 TL072, U2 TL072, U3 LM317_TO-220, U4 LM317_TO-220

Commit message: Uses LM317 for regulators now.
Parts:
- C1, C12, C4, C5: footprint Capacitor_THT:C_Radial_D5.0mm_H11.0mm_P2.00mm -> Capacitor_THT:CP_Radial_D5.0mm_P2.00mm
- C13, C14, C15, C16: LCSC Part # C45669 -> C1710
Changed lines of the file:
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@@
       (effects (font (size 1.27 1.27)) (justify left))
     )
-    (property "Footprint" "Capacitor_THT:C_Radial_D5.0mm_H11.0mm_P2.00mm" (id 2) (at 78.74 179.07 0)
+    (property "Footprint" "Capacitor_THT:CP_Radial_D5.0mm_P2.00mm" (id 2) (at 78.74 179.07 0)
       (effects (font (size 1.27 1.27)) hide)
     )
@@
       (effects (font (size 1.27 1.27)) (justify left))
     )
-    (property "Footprint" "Capacitor_THT:C_Radial_D5.0mm_H11.0mm_P2.00mm" (id 2) (at 60.96 184.15 0)
+    (property "Footprint" "Capacitor_THT:CP_Radial_D5.0mm_P2.00mm" (id 2) (at 60.96 184.15 0)
       (effects (font (size 1.27 1.27)) hide)
     )
@@
       (effects (font (size 1.27 1.27)) (justify left))
     )
-    (property "Footprint" "Capacitor_THT:C_Radial_D5.0mm_H11.0mm_P2.00mm" (id 2) (at 123.825 179.07 0)
+    (property "Footprint" "Capacitor_THT:CP_Radial_D5.0mm_P2.00mm" (id 2) (at 123.825 179.07 0)
       (effects (font (size 1.27 1.27)) hide)
     )
@@
       (effects (font (size 1.27 1.27)) (justify left))
     )
-    (property "Footprint" "Capacitor_THT:C_Radial_D5.0mm_H11.0mm_P2.00mm" (id 2) (at 106.045 184.15 0)
+    (property "Footprint" "Capacitor_THT:CP_Radial_D5.0mm_P2.00mm" (id 2) (at 106.045 184.15 0)
       (effects (font (size 1.27 1.27)) hide)
     )
@@
       (effects (font (size 1.27 1.27)) hide)
     )
-    (property "LCSC Part #" "C45669" (id 5) (at 152.4 25.4 0)
+    (property "LCSC Part #" "C1710" (id 5) (at 152.4 25.4 0)
       (effects (font (size 1.27 1.27)) hide)
     )
@@
       (effects (font (size 1.27 1.27)) hide)
     )
-    (property "LCSC Part #" "C45669" (id 5) (at 152.4 66.04 0)
+    (property "LCSC Part #" "C1710" (id 5) (at 152.4 66.04 0)
       (effects (font (size 1.27 1.27)) hide)
     )
@@
       (effects (font (size 1.27 1.27)) hide)
     )
-    (property "LCSC Part #" "C45669" (id 5) (at 100.33 25.4 0)
+    (property "LCSC Part #" "C1710" (id 5) (at 100.33 25.4 0)
       (effects (font (size 1.27 1.27)) hide)
     )
@@
       (effects (font (size 1.27 1.27)) hide)
     )
-    (property "LCSC Part #" "C45669" (id 5) (at 99.695 66.04 0)
+    (property "LCSC Part #" "C1710" (id 5) (at 99.695 66.04 0)
       (effects (font (size 1.27 1.27)) hide)
     )
@@
     )
     (path "/00000000-0000-0000-0000-00005fc0c3f4"
-      (reference "C1") (unit 1) (value "10uF") (footprint "Capacitor_THT:C_Radial_D5.0mm_H11.0mm_P2.00mm")
+      (reference "C1") (unit 1) (value "10uF") (footprint "Capacitor_THT:CP_Radial_D5.0mm_P2.00mm")
     )
     (path "/00000000-0000-0000-0000-000062324aa8"
@@
     )
     (path "/00000000-0000-0000-0000-00005fb7b8c7"
-      (reference "C4") (unit 1) (value "22uF") (footprint "Capacitor_THT:C_Radial_D5.0mm_H11.0mm_P2.00mm")
+      (reference "C4") (unit 1) (value "22uF") (footprint "Capacitor_THT:CP_Radial_D5.0mm_P2.00mm")
     )
     (path "/3203517d-ed54-4cc4-b113-22afc6338400"
-      (reference "C5") (unit 1) (value "10uF") (footprint "Capacitor_THT:C_Radial_D5.0mm_H11.0mm_P2.00mm")
+      (reference "C5") (unit 1) (value "10uF") (footprint "Capacitor_THT:CP_Radial_D5.0mm_P2.00mm")
     )
     (path "/00000000-0000-0000-0000-000060fb74da"
@@
     )
     (path "/08a1d9e1-6bb3-42f1-9285-4191da62a2df"
-      (reference "C12") (unit 1) (value "22uF") (footprint "Capacitor_THT:C_Radial_D5.0mm_H11.0mm_P2.00mm")
+      (reference "C12") (unit 1) (value "22uF") (footprint "Capacitor_THT:CP_Radial_D5.0mm_P2.00mm")
     )
     (path "/fb87670f-a6c2-4ad7-8373-bff6eeb59357"
